Commit message: Modify LiDAR update rate.
Set rate to 5.

Warning Message:
[async_slam_toolbox_node-9] [INFO] [1697282044.282229935] [slam_toolbox]: Message Filter dropping message: frame 'base_laser' at time 1305.200 for reason 'discarding message because the queue is full'

File: husky_ws/src/husky/LMS1xx/urdf/sick_lms1xx.urdf.xacro (robot description, xacro)
@@ -26,5 +26,5 @@
 -->
 <robot xmlns:xacro="http://www.ros.org/wiki/xacro">
-  <xacro:macro name="sick_lms1xx" params="frame:=laser topic:=scan sample_size:=720 update_rate:=50
+  <xacro:macro name="sick_lms1xx" params="frame:=laser topic:=scan sample_size:=720 update_rate:=5
                min_angle:=-2.35619 max_angle:=2.35619 min_range:=0.1 max_range:=30.0 robot_namespace:=/" >
     <link name="${frame}">
