Commit message: Remove the link in ZED urdf.
We will use the settings provide by the file `zed_macro.urdf.xacro`.

File: zed_ws/src/zed-ros2-wrapper/zed_wrapper/urdf/zed_gazebo.urdf.xacro (robot description, xacro)
@@ -1,81 +1,4 @@
 <?xml version="1.0"?>
 <robot xmlns:xacro="http://ros.org/wiki/xacro">
-  <xacro:property name="baseline" value="0.12"/>
-  <xacro:macro name="zed2"
-               params="link_prefix:=''
-                       joint_prefix:=''">
-    <!-- Camera Center -->
-    <link name="${link_prefix}zed2_camera_center">
-      <inertial>
-        <mass value="0.16140"/>
-        <origin xyz="0 0 0"/>
-        <inertia
-          ixx="0.0003947" ixy="0.0" ixz="3.3365e-8"
-          iyy="2.417e-5" iyz="0.0"
-          izz="0.0003973"/>
-      </inertial>
-      <visual>
-        <geometry>
-          <mesh filename="package://leo_erc_description/models/ZED2.dae"/>
-        </geometry>
-      </visual>
-      <collision>
-        <geometry>
-          <mesh filename="package://leo_erc_description/models/ZED2.dae"/>
-        </geometry>
-      </collision>
-    </link>
-    <!-- Left Camera -->
-    <joint name="${joint_prefix}zed2_left_camera_joint" type="fixed">
-      <parent link="${link_prefix}zed2_camera_center"/>
-      <child link="${link_prefix}zed2_left_camera_frame"/>
-      <origin xyz="0 ${baseline/2} 0" rpy="0 0 0" />
-    </joint>
-    <link name="${link_prefix}zed2_left_camera_frame" />
-    <joint name="${joint_prefix}zed2_left_camera_optical_joint" type="fixed">
-      <origin xyz="0 0 0" rpy="-${pi/2} 0.0 -${pi/2}"/>
-      <parent link="${link_prefix}zed2_left_camera_frame"/>
-      <child link="${link_prefix}zed2_left_camera_optical_frame"/>
-    </joint>
-    <link name="${link_prefix}zed2_left_camera_optical_frame"/>
-    <!-- Right Camera -->
-    <joint name="${joint_prefix}zed2_right_camera_joint" type="fixed">
-      <parent link="${link_prefix}zed2_camera_center"/>
-      <child link="${link_prefix}zed2_right_camera_frame"/>
-      <origin xyz="0 -${baseline/2} 0" rpy="0 0 0" />
-    </joint>
-    <link name="${link_prefix}zed2_right_camera_frame" />
-    <joint name="${joint_prefix}zed2_right_camera_optical_joint" type="fixed">
-      <origin xyz="0 0 0" rpy="-${pi/2} 0.0 -${pi/2}"/>
-      <parent link="${link_prefix}zed2_right_camera_frame"/>
-      <child link="${link_prefix}zed2_right_camera_optical_frame"/>
-    </joint>
-    <link name="${link_prefix}zed2_right_camera_optical_frame"/>
-    <!-- Sensors -->
-    <joint name="${joint_prefix}zed2_mag_joint" type="fixed">
-      <parent link="${link_prefix}zed2_camera_center"/>
-      <child link="${link_prefix}zed2_mag_link"/>
-      <origin xyz="0 0 0" rpy="0 0 0" />
-    </joint>
-    <link name="${link_prefix}zed2_mag_link" />
-    <joint name="${joint_prefix}zed2_baro_joint" type="fixed">
-      <parent link="${link_prefix}zed2_camera_center"/>
-      <child link="${link_prefix}zed2_baro_link"/>
-      <origin xyz="0 0 0" rpy="0 0 0" />
-    </joint>
-    <link name="${link_prefix}zed2_baro_link" />
-    <joint name="${joint_prefix}zed2_temp_left_joint" type="fixed">
-      <parent link="${link_prefix}zed2_left_camera_frame"/>
-      <child link="${link_prefix}zed2_temp_left_link"/>
-      <origin xyz="0 0 0" rpy="0 0 0" />
-    </joint>
-    <link name="${link_prefix}zed2_temp_left_link" />
-    <joint name="${joint_prefix}zed2_temp_right_joint" type="fixed">
-        <parent link="${link_prefix}zed2_right_camera_frame"/>
-        <child link="${link_prefix}zed2_temp_right_link"/>
-        <origin xyz="0 0 0" rpy="0 0 0" />
-    </joint>
-    <link name="${link_prefix}zed2_temp_right_link" />
-  </xacro:macro>
   <xacro:macro name="zed2_gazebo"
                params="robot_ns:=''">
