Commit message: Add the tag `inertial` in ZED urdf.
Gazebo needs the inertial tags for every link. Just as you have <collision> and <visual>, you need to define <inertial>.

Reference: https://answers.gazebosim.org/question/21647

File: zed_ws/src/zed-ros2-wrapper/zed_wrapper/urdf/zed_macro.urdf.xacro (robot description, xacro)
@@ -76,4 +76,9 @@
     <!-- Camera Center -->
     <link name="${name}_camera_center">
+      <inertial>
+        <mass value="0.16140"/>
+        <origin xyz="0 0 0"/>
+        <inertia ixx="0.0003947" ixy="0.0" ixz="3.3365e-8" iyy="2.417e-5" iyz="0.0" izz="0.0003973"/>
+      </inertial>
       <visual>
         <origin xyz="${screw_offset_x} 0 ${screw_offset_z}" rpy="0 0 0"/>
