Commit message: Rename and Re-position the LiDAR
- Modify the position from (-0.064 0 0.122) to (0.002 0.07 0.122)
- Rename the link name from `base_scan` to `base_scan_1`
- Rename the scan topic from `scan` to `scan_1`

File: cartographer_ws/src/multi_lidar/multi_lidar_desp/urdf/turtlebot3_waffle.urdf (robot description, URDF)
Before this commit: robot turtlebot3_waffle, 13 links, 12 joints
Links:
- removed link base_scan
- added link base_scan_1, mass 0.114; collision cylinder length=0.0315 radius=0.055; visual mesh filename=package://turtlebot3_gazebo/models/turtlebot3_common/meshes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 scale=0.001 0.001 0.001
Joints:
- removed joint scan_joint
- added joint scan_joint_1: type fixed, parent base_link, child base_scan_1, origin xyz=0.002 0.07 0.122 rpy=0 0 0

Commit message: Add second LiDAR in URDF and model config
- In URDF:
  - Link: base_scan_2
  - Joint: scan_joint_2
- In model config
  - Link: base_scan_2
  - Joint: lidar_joint_2

Directly copy how the base_link_1 used in the model,
and simply modify to base_link_2.

File: cartographer_ws/src/multi_lidar/multi_lidar_desp/urdf/turtlebot3_waffle.urdf (robot description, URDF)
Before this commit: robot turtlebot3_waffle, 13 links, 12 joints
Links:
- added link base_scan_2, mass 0.114; collision cylinder length=0.0315 radius=0.055; visual mesh filename=package://turtlebot3_gazebo/models/turtlebot3_common/meshes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 scale=0.001 0.001 0.001
Joints:
- added joint scan_joint_2: type fixed, parent base_link, child base_scan_2, origin xyz=-0.16 -0.070 0.122 rpy=0 0 0
