Commit message: Incorporate the ZED urdf into the Husky urdf.
Replace "realsense" with "zed". The remaining part remains the same.

File: zed_to_husky_ws/workspaces/husky_ws/src/husky/husky_description/urdf/accessories/zed/zed_descr.urdf.xacro (robot description, xacro)
@@ -18,8 +18,8 @@
   <xacro:arg name="camera_name"   default="zed" />
   <xacro:arg name="camera_model"  default="zed" />
-  <xacro:include filename="$(find zed_wrapper)/urdf/zed_macro.urdf.xacro" />
+  <xacro:include filename="$(find husky_description)/urdf/accessories/zed/zed_macro.urdf.xacro" />
   <xacro:zed_camera name="$(arg camera_name)" model="$(arg camera_model)">
   </xacro:zed_camera>
-  <xacro:include filename="$(find zed_wrapper)/urdf/zed_gazebo.urdf.xacro" />
+  <xacro:include filename="$(find husky_description)/urdf/accessories/zed/zed_gazebo.urdf.xacro" />
   <xacro:zed_gazebo name="$(arg camera_name)" />
 </robot>

File: zed_to_husky_ws/workspaces/husky_ws/src/husky/husky_description/urdf/accessories/zed/zed_macro.urdf.xacro (robot description, xacro)
@@ -16,5 +16,5 @@
 -->
 <robot xmlns:xacro="http://wiki.ros.org/xacro">
-  <xacro:include filename="$(find zed_wrapper)/urdf/include/materials.urdf.xacro" />
+  <xacro:include filename="$(find husky_description)/urdf/accessories/zed/include/materials.urdf.xacro" />
   <xacro:property name="M_PI"     value="3.1415926535897931" />
   <!--
@@ -85,5 +85,5 @@
         <origin xyz="${screw_offset_x} 0 ${screw_offset_z}" rpy="0 0 0"/>
         <geometry>
-          <mesh filename="package://zed_interfaces/meshes/${model}.stl" />
+          <mesh filename="package://husky_description/meshes/accessories/zed/${model}.stl" />
         </geometry>
         <material name="${model}_mat" />
@@ -91,5 +91,5 @@
       <collision>
         <geometry>
-          <mesh filename="package://zed_interfaces/meshes/${model}.stl" />
+          <mesh filename="package://husky_description/meshes/accessories/zed/${model}.stl" />
         </geometry>
       </collision>

File: zed_to_husky_ws/workspaces/husky_ws/src/husky/husky_description/urdf/husky_macro.urdf.xacro (robot description, xacro)
@@ -4,8 +4,10 @@
   <xacro:arg name="laser_xyz" default="$(optenv CPR_LASER_XYZ 0.2206 0.0 0.00635)" />
   <xacro:arg name="laser_rpy" default="$(optenv CPR_LASER_RPY 0.0 0.0 0.0)" />
-  <xacro:arg name="realsense_enabled" default="$(optenv CPR_REALSENSE 0)" />
-  <xacro:arg name="realsense_xyz" default="$(optenv CPR_REALSENSE_XYZ 0 0 0)" />
-  <xacro:arg name="realsense_rpy" default="$(optenv CPR_REALSENSE_RPY 0 0 0)" />
-  <xacro:arg name="realsense_mount" default="$(optenv CPR_REALSENSE_MOUNT_FRAME sensor_arch_mount_link)" />
+  <xacro:arg name="zed_enabled" default="0" />
+  <xacro:arg name="zed_xyz" default="0 0 0" />
+  <xacro:arg name="zed_rpy" default="0 0 3.14" />
+  <xacro:arg name="zed_mount" default="sensor_arch_mount_link" />
+  <xacro:arg name="camera_name"   default="zed" />
+  <xacro:arg name="camera_model"  default="zed2i" />
   <xacro:property name="husky_front_bumper_extend" value="$(optenv HUSKY_FRONT_BUMPER_EXTEND 0)" />
   <xacro:property name="husky_rear_bumper_extend" value="$(optenv HUSKY_REAR_BUMPER_EXTEND 0)" />
@@ -16,7 +18,8 @@
   <xacro:include filename="$(find husky_description)/urdf/decorations.urdf.xacro" />
   <xacro:include filename="$(find husky_description)/urdf/wheel.urdf.xacro" />
-  <xacro:include filename="$(find husky_description)/urdf/accessories/intel_realsense.urdf.xacro"/>
   <xacro:include filename="$(find husky_description)/urdf/accessories/sick_lms1xx_mount.urdf.xacro"/>
   <xacro:include filename="$(find husky_description)/urdf/accessories/sensor_arch.urdf.xacro"/>
+  <xacro:include filename="$(find husky_description)/urdf/accessories/zed/zed_macro.urdf.xacro" />
+  <xacro:include filename="$(find husky_description)/urdf/accessories/zed/zed_gazebo.urdf.xacro" />
   <xacro:property name="M_PI" value="3.14159"/>
   <xacro:macro name="husky" params="prefix">
@@ -113,23 +116,25 @@
     </xacro:if>
     <!--
-      top sensor arch; include this if we have realsense enabled
+      top sensor arch; include this if we have zed enabled
       keep this as a property to make it easier to add multiple conditions, should we need
       the top bar for any additional sensors in the future
     -->
-    <xacro:property name="topbar_needed_realsense" value="$(arg realsense_enabled)" />
-    <xacro:if value="${topbar_needed_realsense}">
+    <xacro:property name="topbar_needed_zed" value="$(arg zed_enabled)" />
+    <xacro:if value="${topbar_needed_zed}">
         <xacro:sensor_arch prefix="" parent="top_plate_link">
             <origin xyz="-0.35 0 0.51" rpy="0 0 -3.14"/>
         </xacro:sensor_arch>
     </xacro:if>
-    <!-- add the intel realsense to the topbar if needed -->
-    <xacro:if value="$(arg realsense_enabled)">
-      <link name="realsense_mountpoint"/>
-      <joint name="realsense_mountpoint_joint" type="fixed">
-        <origin xyz="$(arg realsense_xyz)" rpy="$(arg realsense_rpy)" />
-        <parent link="$(arg realsense_mount)"/>
-        <child link="realsense_mountpoint" />
+    <!-- add the stereolab zed to the topbar if needed -->
+    <xacro:if value="$(arg zed_enabled)">
+      <joint name="zed_mountpoint_joint" type="fixed">
+        <origin xyz="$(arg zed_xyz)" rpy="$(arg zed_rpy)" />
+        <parent link="$(arg zed_mount)"/>
+        <child link="$(arg camera_name)_camera_link" />
       </joint>
-      <xacro:intel_realsense_mount prefix="camera" topic="realsense" parent_link="realsense_mountpoint"/>
+      <xacro:zed_camera name="$(arg camera_name)" model="$(arg camera_model)" />
+      <xacro:if value="$(arg is_sim)">
+        <xacro:zed_gazebo name="$(arg camera_name)" />
+      </xacro:if>
     </xacro:if>
     <ros2_control name="${prefix}husky_hardware" type="system">
