Commit message: Include VLP16 LiDAR model into husky description
- Set parent to `top_plate_link` which is a plate on top of the husky

File: vlp_to_husky_ws/workspaces/husky_ws/src/husky/husky_description/urdf/husky.urdf.xacro (robot description, xacro)
@@ -5,5 +5,10 @@
   <xacro:arg name="prefix" default="" />
   <xacro:arg name="gazebo_controllers" default="$(find husky_control)/config/control.yaml" />
+  <xacro:arg name="gpu" default="false"/>
+  <xacro:arg name="organize_cloud" default="false"/>
+  <xacro:property name="gpu" value="$(arg gpu)" />
+  <xacro:property name="organize_cloud" value="$(arg organize_cloud)" />
   <xacro:include filename="$(find husky_description)/urdf/husky_macro.urdf.xacro" />
+  <xacro:include filename="$(find velodyne_description)/urdf/VLP-16.urdf.xacro"/>
   <!-- Load husky description -->
   <xacro:husky prefix="$(arg prefix)" />
@@ -43,3 +48,7 @@
   <!-- Optional custom includes. -->
   <xacro:include filename="$(arg urdf_extras)" />
+  <!-- Add LiDAR model -->
+  <xacro:VLP-16 parent="top_plate_link" name="velodyne" topic="/velodyne_points" organize_cloud="${organize_cloud}" hz="10" samples="440" gpu="${gpu}">
+    <origin xyz="0.25 0 0.0" rpy="0 0 0" />
+  </xacro:VLP-16>
 </robot>
