Commit message: Fix mesh file not found
It seems that the package URL description before is not working since we didn't set the model config in velodyne_description.
Instead of setting model config, I think it is faster if we directly change to find command

File: vlp_to_husky_ws/workspaces/husky_ws/src/velodyne_simulator/velodyne_description/urdf/VLP-16.urdf.xacro (robot description, xacro)
@@ -18,10 +18,10 @@
       <visual>
         <geometry>
-          <mesh filename="package://velodyne_description/meshes/VLP16_base_1.dae" />
+          <mesh filename="$(find velodyne_description)/meshes/VLP16_base_1.dae" />
         </geometry>
       </visual>
       <visual>
         <geometry>
-          <mesh filename="package://velodyne_description/meshes/VLP16_base_2.dae" />
+          <mesh filename="$(find velodyne_description)/meshes/VLP16_base_2.dae" />
         </geometry>
       </visual>
@@ -47,5 +47,5 @@
         <origin xyz="0 0 -0.0377" />
         <geometry>
-          <mesh filename="package://velodyne_description/meshes/VLP16_scan.dae" />
+          <mesh filename="$(find velodyne_description)/meshes/VLP16_scan.dae" />
         </geometry>
       </visual>
