Commit message: Modify Husky's description.
Uncomment the settings in urdf to support laser_enabled and realsense_enabled.

File: husky_ws/src/husky/husky_description/urdf/husky_macro.urdf.xacro (robot description, xacro)
@@ -17,5 +17,5 @@
   <xacro:include filename="$(find husky_description)/urdf/wheel.urdf.xacro" />
   <xacro:include filename="$(find husky_description)/urdf/accessories/intel_realsense.urdf.xacro"/>
-  <!-- <xacro:include filename="$(find husky_description)/urdf/accessories/sick_lms1xx_mount.urdf.xacro"/> -->
+  <xacro:include filename="$(find husky_description)/urdf/accessories/sick_lms1xx_mount.urdf.xacro"/>
   <xacro:include filename="$(find husky_description)/urdf/accessories/sensor_arch.urdf.xacro"/>
   <xacro:property name="M_PI" value="3.14159"/>
@@ -103,13 +103,13 @@
     </xacro:husky_wheel>
     <xacro:husky_decorate />
-    <!-- <xacro:if value="$(arg laser_enabled)">
-      <xacro:sick_lms1xx_mount prefix="base"/>
-      <xacro:sick_lms1xx frame="base_laser" topic="scan" robot_namespace="$(arg robot_namespace)"/>
-      <joint name="laser_mount_joint" type="fixed">
-        <origin xyz="$(arg laser_xyz)" rpy="$(arg laser_rpy)" />
-        <parent link="top_plate_link" />
-        <child link="base_laser_mount" />
-      </joint>
-    </xacro:if> -->
+    <xacro:if value="$(arg laser_enabled)">
+        <xacro:sick_lms1xx_mount prefix="base"/>
+        <xacro:sick_lms1xx frame="base_laser" topic="scan" robot_namespace="$(arg robot_namespace)"/>
+        <joint name="laser_mount_joint" type="fixed">
+            <origin xyz="$(arg laser_xyz)" rpy="$(arg laser_rpy)" />
+            <parent link="top_plate_link" />
+            <child link="base_laser_mount" />
+        </joint>
+    </xacro:if>
     <!--
       top sensor arch; include this if we have realsense enabled
@@ -117,10 +117,10 @@
       the top bar for any additional sensors in the future
     -->
-    <!-- <xacro:property name="topbar_needed_realsense" value="$(arg realsense_enabled)" />
+    <xacro:property name="topbar_needed_realsense" value="$(arg realsense_enabled)" />
     <xacro:if value="${topbar_needed_realsense}">
-      <xacro:sensor_arch prefix="" parent="top_plate_link">
-        <origin xyz="-0.35 0 0.51" rpy="0 0 -3.14"/>
-      </xacro:sensor_arch>
-    </xacro:if> -->
+        <xacro:sensor_arch prefix="" parent="top_plate_link">
+            <origin xyz="-0.35 0 0.51" rpy="0 0 -3.14"/>
+        </xacro:sensor_arch>
+    </xacro:if>
     <!-- add the intel realsense to the topbar if needed -->
     <xacro:if value="$(arg realsense_enabled)">

Commit message: Fix the wheelbase in husky urdf.
This pertains to the wheel separation distance, ideally set at 0.545m according to the technical specifications. However, within the clearpath_common configuration for Husky, it's designated 0.555m. I've opted to follow the clearpath_common.

Reference:
- https://clearpathrobotics.com/husky-unmanned-ground-vehicle-robot/
- https://github.com/clearpathrobotics/clearpath_common/blob/4f5456a26e4769e6c9d40aa0b733f56ad1e68a1b/clearpath_control/config/a200/control.yaml#L16

File: husky_ws/src/husky/husky_description/urdf/husky_macro.urdf.xacro (robot description, xacro)
@@ -26,5 +26,5 @@
     <xacro:property name="base_z_size" value="0.24750000" />
     <!-- Wheel Mounting Positions -->
-    <xacro:property name="wheelbase" value="0.5120" />
+    <xacro:property name="wheelbase" value="0.5550" />
     <xacro:property name="track" value="0.5708" />
     <xacro:property name="wheel_vertical_offset" value="0.03282" />
