Commit message: Modify the VLP-16 position and change default map.
Lowering the LiDAR height for TurtleBot3's small-scale environment may enhance data quality.

File: kobuki_ws/src/kobuki_ros/kobuki_description/urdf/kobuki_VLP16.urdf.xacro (robot description, xacro)
@@ -18,5 +18,5 @@
         <xacro:include filename="$(find velodyne_description)/urdf/VLP-16.urdf.xacro"/>
         <xacro:VLP-16 is_sim="${is_sim}" parent="base_link" name="velodyne" topic="/velodyne_points" organize_cloud="${organize_cloud}" hz="10" samples="440" gpu="${gpu}">
-            <origin xyz="0 0 0.4" rpy="0 0 0" />
+            <origin xyz="0 0 0.2" rpy="0 0 0" />
         </xacro:VLP-16>
     </xacro:if>
