Commit message: feat(turtlebot3_ws): Publish lidar scan and point cloud through OmniGraph
Refs:
- http://wiki.ros.org/urdf/XML/sensor
- https://github.com/isaac-sim/urdf-importer-extension/blob/b161d55f4bcabe266b8db6707b5c2768aedcde21/source/extensions/omni.importer.urdf/data/urdf/tests/test_sensor.urdf#L60-L72
- https://docs.omniverse.nvidia.com/isaacsim/latest/features/sensors_simulation/isaac_sim_sensors_rtx_based_lidar.html

File: turtlebot3_ws/src/turtlebot3/turtlebot3_description/urdf/turtlebot3_burger_isaacsim.urdf.xacro (robot description, xacro)
@@ -168,3 +168,11 @@
     </camera>
   </sensor>
+  <sensor name="lidar" type="ray" update_rate="30" isaac_sim_config="Example_Solid_State">
+    <parent link="base_scan"/>
+    <origin xyz="0 0 0" rpy="0 0 0"/>
+    <ray>
+      <horizontal samples="21" resolution="1" min_angle="-0.785398" max_angle="0.785398"/>
+      <vertical samples="20" resolution="1" min_angle="-0.523599" max_angle="0.523599"/>
+    </ray>
+  </sensor>
 </robot>
