Commit message: feat(go2_ws): Update Go2 urdf model.
The `xacro/robot.xacro` and `urdf/go2_description.urdf` are not synchronized, such as the position of IMU is different, there is no head and radar in `robot.xacro`. Based on experience, the urdf is closer to real robot, so `robot.xacro` is updated to be the same as `go2_description.urdf`.

The gazebo plugin is not updated yet.

Note: For easy reading, I rearranged the link and joint order in the order of link first and then joint. In addition, the original `robot.xacro` has been formatted; I formatted it again after modification. Since the difference is not very large, I merged it into one commit directly.

File: go2_ws/src/go2_description/xacro/leg.xacro (robot description, xacro)
@@ -1,5 +1,4 @@
 <?xml version="1.0"?>
 <robot xmlns:xacro="http://www.ros.org/wiki/xacro">
-    <xacro:include filename="$(find go2_description)/xacro/transmission.xacro"/>
     <xacro:macro name="leg" params="name mirror mirror_dae front_hind front_hind_dae">
         <joint name="${name}_hip_joint" type="revolute">
@@ -16,5 +15,5 @@
                 <origin rpy="0 0 0" xyz="${-leg_offset_x} ${leg_offset_y} 0"/>
             </xacro:if>
-            <parent link="trunk"/>
+            <parent link="base_link"/>
             <child link="${name}_hip"/>
             <axis xyz="1 0 0"/>
@@ -55,8 +54,5 @@
                 <origin rpy="0 0 0" xyz="${hip_com_x*front_hind} ${hip_com_y*mirror} ${hip_com_z}"/>
                 <mass value="${hip_mass}"/>
-                <inertia
-                    ixx="${hip_ixx}" ixy="${hip_ixy*mirror*front_hind}" ixz="${hip_ixz*front_hind}"
-                    iyy="${hip_iyy}" iyz="${hip_iyz*mirror}"
-                    izz="${hip_izz}"/>
+                <inertia ixx="${hip_ixx}" ixy="${hip_ixy*mirror*front_hind}" ixz="${hip_ixz*front_hind}" iyy="${hip_iyy}" iyz="${hip_iyz*mirror}" izz="${hip_izz}"/>
             </inertial>
         </link>
@@ -91,8 +87,5 @@
                 <origin rpy="0 0 0" xyz="${thigh_com_x} ${thigh_com_y*mirror} ${thigh_com_z}"/>
                 <mass value="${thigh_mass}"/>
-                <inertia
-                    ixx="${thigh_ixx}" ixy="${thigh_ixy*mirror}" ixz="${thigh_ixz}"
-                    iyy="${thigh_iyy}" iyz="${thigh_iyz*mirror}"
-                    izz="${thigh_izz}"/>
+                <inertia ixx="${thigh_ixx}" ixy="${thigh_ixy*mirror}" ixz="${thigh_ixz}" iyy="${thigh_iyy}" iyz="${thigh_iyz*mirror}" izz="${thigh_izz}"/>
             </inertial>
         </link>
@@ -122,11 +115,8 @@
                 <origin rpy="0 0 0" xyz="${calf_com_x} ${calf_com_y} ${calf_com_z}"/>
                 <mass value="${calf_mass}"/>
-                <inertia
-                    ixx="${calf_ixx}" ixy="${calf_ixy}" ixz="${calf_ixz}"
-                    iyy="${calf_iyy}" iyz="${calf_iyz}"
-                    izz="${calf_izz}"/>
+                <inertia ixx="${calf_ixx}" ixy="${calf_ixy}" ixz="${calf_ixz}" iyy="${calf_iyy}" iyz="${calf_iyz}" izz="${calf_izz}"/>
             </inertial>
         </link>
-        <joint name="${name}_foot_fixed" type="fixed">0
+        <joint name="${name}_foot_joint" type="fixed">
             <origin rpy="0 0 0" xyz="0 0 ${-(calf_length)}"/>
             <parent link="${name}_calf"/>
@@ -149,11 +139,7 @@
             <inertial>
                 <mass value="${foot_mass}"/>
-                <inertia
-                    ixx="${(2*foot_mass)/5.0*(foot_radius*foot_radius)}" ixy="0.0" ixz="0.0"
-                    iyy="${(2*foot_mass)/5.0*(foot_radius*foot_radius)}" iyz="0.0"
-                    izz="${(2*foot_mass)/5.0*(foot_radius*foot_radius)}"/>
+                <inertia ixx="${(2*foot_mass)/5.0*(foot_radius*foot_radius)}" ixy="0.0" ixz="0.0" iyy="${(2*foot_mass)/5.0*(foot_radius*foot_radius)}" iyz="0.0" izz="${(2*foot_mass)/5.0*(foot_radius*foot_radius)}"/>
             </inertial>
         </link>
-        <xacro:leg_transmission name="${name}"/>
     </xacro:macro>
 </robot>

File: go2_ws/src/go2_description/xacro/robot.xacro (robot description, xacro)
@@ -1,36 +1,26 @@
 <?xml version="1.0"?>
-<robot name="go2" xmlns:xacro="http://www.ros.org/wiki/xacro">
-    <xacro:arg name="DEBUG" default="false"/>
+<robot name="go2"
+    xmlns:xacro="http://www.ros.org/wiki/xacro">
+    <!-- Declare argument -->
+    <xacro:arg name="enable_gazebo" default="False"/>
+    <!-- Declare parameters -->
+    <xacro:property name="enable_gazebo" value="$(arg enable_gazebo)"/>
+    <!-- Include other file -->
     <xacro:include filename="$(find go2_description)/xacro/const.xacro"/>
     <xacro:include filename="$(find go2_description)/xacro/materials.xacro"/>
     <xacro:include filename="$(find go2_description)/xacro/leg.xacro"/>
-    <!-- <xacro:include filename="$(find go2_description)/xacro/stairs.xacro"/> -->
-    <xacro:include filename="$(find go2_description)/xacro/gazebo.xacro"/>
-    <!-- <xacro:include filename="$(find go2_gazebo)/launch/stairs.urdf.xacro"/> -->
-    <!-- <xacro:stairs stairs="15" xpos="0" ypos="0" zpos="0" /> -->
-    <!-- Rotor related joint and link is only for demonstrate location. -->
-    <!-- Actually, the rotor will rotate and the joint is not fixed. Reduction ratio should be considered. -->
-    <!-- Debug mode will hung up the robot, use "true" or "false" to switch it. -->
-    <xacro:if value="$(arg DEBUG)">
-        <link name="world"/>
-        <joint name="base_static_joint" type="fixed">
-            <origin rpy="0 0 0" xyz="0 0 0"/>
-            <parent link="world"/>
-            <child link="base_link"/>
-        </joint>
+    <xacro:if value="${enable_gazebo}">
+        <xacro:include filename="$(find go2_description)/xacro/gazebo.xacro"/>
     </xacro:if>
-    <link name="base_link">
-        <visual>
-            <origin rpy="0 0 0" xyz="0 0 0"/>
-            <geometry>
-                <box size="0.001 0.001 0.001"/>
-            </geometry>
-        </visual>
-    </link>
-    <joint name="floating_base" type="fixed">
-        <origin rpy="0 0 0" xyz="0 0 0"/>
+    <!-- base_link -->
+    <link name="base_link"/>
+    <!-- base_footprint -->
+    <link name="base_footprint"/>
+    <joint name="base_footprint_joint" type="fixed">
         <parent link="base_link"/>
-        <child link="trunk"/>
+        <child link="base_footprint"/>
+        <origin xyz="0 0 0" rpy="0 0 0"/>
     </joint>
+    <!-- trunk -->
     <link name="trunk">
         <visual>
@@ -39,5 +29,4 @@
                 <mesh filename="package://go2_description/meshes/trunk.dae" scale="1 1 1"/>
             </geometry>
-            <!-- <material name="orange"/> -->
         </visual>
         <collision>
@@ -50,64 +39,80 @@
             <origin rpy="0 0 0" xyz="${trunk_com_x} ${trunk_com_y} ${trunk_com_z}"/>
             <mass value="${trunk_mass}"/>
-            <inertia
-                ixx="${trunk_ixx}" ixy="${trunk_ixy}" ixz="${trunk_ixz}"
-                iyy="${trunk_iyy}" iyz="${trunk_iyz}"
-                izz="${trunk_izz}"/>
+            <inertia ixx="${trunk_ixx}" ixy="${trunk_ixy}" ixz="${trunk_ixz}" iyy="${trunk_iyy}" iyz="${trunk_iyz}" izz="${trunk_izz}"/>
         </inertial>
     </link>
-    <joint name="imu_joint" type="fixed">
-        <parent link="trunk"/>
-        <child link="imu_link"/>
+    <joint name="floating_base" type="fixed">
         <origin rpy="0 0 0" xyz="0 0 0"/>
+        <parent link="base_link"/>
+        <child link="trunk"/>
     </joint>
-    <link name="imu_link">
+    <!-- Include four legs -->
+    <xacro:leg name="FR" mirror="-1" mirror_dae= "False" front_hind="1" front_hind_dae="True" />
+    <xacro:leg name="FL" mirror="1" mirror_dae="True" front_hind="1" front_hind_dae="True" />
+    <xacro:leg name="RR" mirror="-1" mirror_dae="False" front_hind="-1" front_hind_dae="False" />
+    <xacro:leg name="RL" mirror="1" mirror_dae="True" front_hind="-1" front_hind_dae="False" />
+    <!-- Head_upper -->
+    <link name="Head_upper">
         <inertial>
-            <mass value="0.001"/>
-            <origin rpy="0 0 0" xyz="0 0 0"/>
-            <inertia ixx="0.0001" ixy="0" ixz="0" iyy="0.0001" iyz="0" izz="0.0001"/>
+            <origin xyz="0 0 0" rpy="0 0 0" />
+            <mass value="0.001" />
+            <inertia ixx="9.6e-06" ixy="0" ixz="0" iyy="9.6e-06" iyz="0" izz="9.6e-06" />
         </inertial>
-        <visual>
-            <origin rpy="0 0 0" xyz="0 0 0"/>
+        <collision>
+            <origin xyz="0 0 0" rpy="0 0 0" />
             <geometry>
-                <box size="0.001 0.001 0.001"/>
-            </geometry>
-            <!-- <material name="red"/> -->
-        </visual>
-        <collision>
-            <origin rpy="0 0 0" xyz="0 0 0"/>
-            <geometry>
-                <box size=".001 .001 .001"/>
+                <cylinder radius="0.05" length="0.09" />
             </geometry>
         </collision>
     </link>
-    <!--
-    <joint name="load_joint" type="fixed">
-        <parent link="trunk"/>
-        <child link="load_link"/>
-        <origin rpy="0 0 0" xyz="0 0 0"/>
+    <joint name="Head_upper_joint" type="fixed" dont_collapse="true">
+        <origin xyz="0.285 0 0.01" rpy="0 0 0" />
+        <parent link="base_link" />
+        <child link="Head_upper" />
+        <axis xyz="0 0 0" />
     </joint>
-    <link name="load_link">
+    <!-- Head_lower -->
+    <link name="Head_lower">
         <inertial>
-            <mass value="5"/>
-            <origin rpy="0 0 0" xyz="0 0 0"/>
-            <inertia ixx="0.01" ixy="0" ixz="0" iyy="0.01" iyz="0" izz="0.01"/>
+            <origin xyz="0 0 0" rpy="0 0 0" />
+            <mass value="0.001" />
+            <inertia ixx="9.6e-06" ixy="0" ixz="0" iyy="9.6e-06" iyz="0" izz="9.6e-06" />
         </inertial>
-        <visual>
-            <origin rpy="0 0 0" xyz="0 0 0.2"/>
+        <collision>
+            <origin xyz="0 0 0" rpy="0 0 0" />
             <geometry>
-                <box size="0.5 0.3 0.2"/>
-            </geometry>
-        </visual>
-        <collision>
-            <origin rpy="0 0 0" xyz="0 0 0"/>
-            <geometry>
-                <box size=".001 .001 .001"/>
+                <sphere radius="0.047" />
             </geometry>
         </collision>
     </link>
--->
-    <xacro:leg name="FR" mirror="-1" mirror_dae= "False" front_hind="1"  front_hind_dae="True"  />
-    <xacro:leg name="FL" mirror="1"  mirror_dae="True"   front_hind="1"  front_hind_dae="True"  />
-    <xacro:leg name="RR" mirror="-1" mirror_dae="False"  front_hind="-1" front_hind_dae="False" />
-    <xacro:leg name="RL" mirror="1"  mirror_dae="True"   front_hind="-1" front_hind_dae="False" />
+    <joint name="Head_lower_joint" type="fixed" dont_collapse="true">
+        <origin xyz="0.008 0 -0.07" rpy="0 0 0" />
+        <parent link="Head_upper" />
+        <child link="Head_lower" />
+        <axis xyz="0 0 0" />
+    </joint>
+    <!-- imu_link -->
+    <link name="imu_link"/>
+    <joint name="imu_joint" type="fixed">
+        <origin xyz="-0.02557 0 0.04232" rpy="0 0 0" />
+        <parent link="base_link" />
+        <child link="imu_link" />
+        <axis xyz="0 0 0" />
+    </joint>
+    <!-- radar -->
+    <link name="radar_link"/>
+    <joint name="radar_joint" type="fixed">
+        <origin xyz="0.28945 0 -0.046825" rpy="0 2.8782 0" />
+        <parent link="base_link" />
+        <child link="radar_link" />
+        <axis xyz="0 0 0" />
+    </joint>
+    <!-- front camera -->
+    <link name="front_camera_link"/>
+    <joint name="front_camera_joint" type="fixed">
+        <origin xyz="0.045 0 0.03" rpy="-1.5708 0 -1.5708" />
+        <parent link="Head_upper" />
+        <child link="front_camera_link" />
+        <axis xyz="0 0 0" />
+    </joint>
 </robot>
