Commit message: feat(go2_ws): Upgrade the `go2_description` to ROS2 humble.
The package provided by Unitree is ros1 noetic, upgrade the related file to ros2 humble.

File: go2_ws/src/go2_description/xacro/robot.xacro (robot description, xacro)
@@ -17,8 +17,8 @@
             <origin rpy="0 0 0" xyz="0 0 0"/>
             <parent link="world"/>
-            <child link="base"/>
+            <child link="base_link"/>
         </joint>
     </xacro:if>
-    <link name="base">
+    <link name="base_link">
         <visual>
             <origin rpy="0 0 0" xyz="0 0 0"/>
@@ -30,5 +30,5 @@
     <joint name="floating_base" type="fixed">
         <origin rpy="0 0 0" xyz="0 0 0"/>
-        <parent link="base"/>
+        <parent link="base_link"/>
         <child link="trunk"/>
     </joint>

Commit message: feat(go2_ws): Remove `trunk` frame in the xacro file.
Since the `trunk` frame is completely redundant, we remove it and move its settings to `base_link`.

Reference: https://github.com/j3soon/ros2-essentials/pull/85#discussion_r2205286058

File: go2_ws/src/go2_description/xacro/robot.xacro (robot description, xacro)
@@ -14,14 +14,7 @@
     </xacro:if>
     <!-- base_link -->
-    <link name="base_link"/>
-    <!-- base_footprint -->
-    <link name="base_footprint"/>
-    <joint name="base_footprint_joint" type="fixed">
-        <parent link="base_link"/>
-        <child link="base_footprint"/>
-        <origin xyz="0 0 0" rpy="0 0 0"/>
-    </joint>
-    <!-- trunk -->
-    <link name="trunk">
+    <!-- Note: Since the `trunk` frame is completely redundant, -->
+    <!--       we remove it and move its settings to `base_link`. -->
+    <link name="base_link">
         <visual>
             <origin rpy="0 0 0" xyz="0 0 0"/>
@@ -42,8 +35,12 @@
         </inertial>
     </link>
-    <joint name="floating_base" type="fixed">
-        <origin rpy="0 0 0" xyz="0 0 0"/>
+    <!-- base_footprint -->
+    <!-- Note: The `base_footprint` link is initially set at `base_link`, -->
+    <!--       but it will be updated based on the actual body height computed using forward kinematics. -->
+    <link name="base_footprint"/>
+    <joint name="base_footprint_joint" type="fixed">
         <parent link="base_link"/>
-        <child link="trunk"/>
+        <child link="base_footprint"/>
+        <origin xyz="0 0 0" rpy="0 0 0"/>
     </joint>
     <!-- Include four legs -->
