Commit message: fix: adjust realsense d435 pose and mesh path for turtlebot3 burger     - adjusted the pose of the Realsense D435 camera in both the SDF and URDF files to ensure correct orientation and positioning on the TurtleBot3 Burger model.         - source: https://github.com/issaiass/realsense2_description

File: template_ws/src/realsense_examples/realsense_desp/urdf/turtlebot3_burger.urdf (robot description, URDF)
Before this commit: robot turtlebot3_burger, 17 links, 16 joints
Joints:
- joint camera_joint: origin xyz=0.2 0 0.172 rpy=0 0 0 -> xyz=-0.02 0 0.201 rpy=0 0 0
