Commit message: feat(stretch3_ws): Modify URDF for Isaac Sim
- `base_link_collision.STL` is an overly large cuboid, which will overlap with the wheel meshes. Changed to visual mesh for better collision mesh.
- `link_{left|right}_wheel_collision.STL` are also cuboids, which will cause bouncing behavior if not modified (think of square wheels)
  Using visual mesh as base_link is not preferred since it will still result in non-smooth mesh (think polygon instead of circle). The preferred way is to directly specify a cylinder as collider, the radius/length/offset follows those of the official stretch 3 USD file.

Screenshots, recording, and references will be attached in PR description

File: stretch3_ws/src/stretch_urdf/stretch_urdf/SE3/stretch_description_SE3_eoa_wrist_dw3_tool_sg3_isaac.urdf (robot description, URDF)
Before this commit: robot stretch, 61 links, 60 joints
Links:
- link base_link: geometry collision mesh filename=./meshes/base_link.STL; visual mesh filename=./meshes/base_link.STL
- link link_left_wheel: geometry collision cylinder length=0.025 radius=0.05; visual mesh filename=./meshes/link_left_wheel.STL
- link link_right_wheel: geometry collision cylinder length=0.025 radius=0.05; visual mesh filename=./meshes/link_right_wheel.STL
