Commit message: feat(ur5_ws): Disable internal collision checking for the gripper.

File: ur5_ws/src/Universal_Robots_ROS2_Driver/ur_moveit_config/srdf/ur.srdf.xacro (robot description, xacro)
@@ -5,5 +5,6 @@
   <!-- parameters -->
   <xacro:arg name="prefix" default="" />
+  <xacro:arg name="use_rg2_gripper" default="true" />
   <xacro:include filename="$(find ur_moveit_config)/srdf/ur_macro.srdf.xacro"/>
-  <xacro:ur_srdf name="$(arg name)" prefix="$(arg prefix)"/>
+  <xacro:ur_srdf name="$(arg name)" prefix="$(arg prefix)" use_rg2_gripper="$(arg use_rg2_gripper)"/>
 </robot>

File: ur5_ws/src/Universal_Robots_ROS2_Driver/ur_moveit_config/srdf/ur_macro.srdf.xacro (robot description, xacro)
@@ -5,5 +5,5 @@
     A URDF file must exist for this robot as well, where the joints and the links that are referenced are defined
 -->
-  <xacro:macro name="ur_srdf" params="name prefix">
+  <xacro:macro name="ur_srdf" params="name prefix use_rg2_gripper">
     <!--GROUPS - Representation of a set of joints and links. This can be useful for specifying DOF to plan for, defining arms, end effectors, etc-->
     <!--LINKS - When a link is specified, the parent joint of that link (if it exists) is automatically included-->
@@ -12,5 +12,11 @@
     <!--SUBGROUPS - Groups can also be formed by referencing to already defined group names-->
     <group name="${prefix}${name}_manipulator">
-      <chain base_link="${prefix}base_link" tip_link="${prefix}tool0" />
+      <!-- With gripper: tip at rg2_base_link; without: tip at tool0-->
+      <xacro:if value="${use_rg2_gripper}">
+        <chain base_link="${prefix}base_link" tip_link="${prefix}rg2_base_link" />
+      </xacro:if>
+      <xacro:if value="${not use_rg2_gripper}">
+        <chain base_link="${prefix}base_link" tip_link="${prefix}tool0" />
+      </xacro:if>
     </group>
     <!--GROUP STATES - Purpose - Define a named state for a particular group, in terms of joint values. This is useful to define states like 'folded arms'-->
@@ -53,4 +59,38 @@
     <disable_collisions link1="${prefix}wrist_1_link" link2="${prefix}wrist_3_link" reason="Never" />
     <disable_collisions link1="${prefix}wrist_2_link" link2="${prefix}wrist_3_link" reason="Adjacent" />
+    <!-- RG2 gripper collision exclusions -->
+    <xacro:if value="${use_rg2_gripper}">
+      <disable_collisions link1="${prefix}rg2_base_link" link2="${prefix}wrist_3_link" reason="Never" />
+      <disable_collisions link1="${prefix}rg2_base_link" link2="${prefix}rg2_hand_link" reason="Adjacent" />
+      <disable_collisions link1="${prefix}rg2_base_link" link2="${prefix}rg2_l_moment_arm_link" reason="Never" />
+      <disable_collisions link1="${prefix}rg2_base_link" link2="${prefix}rg2_r_moment_arm_link" reason="Never" />
+      <disable_collisions link1="${prefix}rg2_base_link" link2="${prefix}rg2_l_finger_link" reason="Never" />
+      <disable_collisions link1="${prefix}rg2_base_link" link2="${prefix}rg2_r_finger_link" reason="Never" />
+      <disable_collisions link1="${prefix}rg2_base_link" link2="${prefix}rg2_l_truss_arm_link" reason="Never" />
+      <disable_collisions link1="${prefix}rg2_base_link" link2="${prefix}rg2_r_truss_arm_link" reason="Never" />
+      <disable_collisions link1="${prefix}rg2_hand_link" link2="${prefix}wrist_3_link" reason="Never" />
+      <disable_collisions link1="${prefix}rg2_hand_link" link2="${prefix}tool0" reason="Never" />
+      <disable_collisions link1="${prefix}rg2_hand_link" link2="${prefix}rg2_l_moment_arm_link" reason="Adjacent" />
+      <disable_collisions link1="${prefix}rg2_hand_link" link2="${prefix}rg2_r_moment_arm_link" reason="Adjacent" />
+      <disable_collisions link1="${prefix}rg2_hand_link" link2="${prefix}rg2_l_truss_arm_link" reason="Adjacent" />
+      <disable_collisions link1="${prefix}rg2_hand_link" link2="${prefix}rg2_r_truss_arm_link" reason="Adjacent" />
+      <disable_collisions link1="${prefix}rg2_hand_link" link2="${prefix}rg2_l_finger_link" reason="Never" />
+      <disable_collisions link1="${prefix}rg2_hand_link" link2="${prefix}rg2_r_finger_link" reason="Never" />
+      <disable_collisions link1="${prefix}rg2_l_moment_arm_link" link2="${prefix}rg2_l_finger_link" reason="Adjacent" />
+      <disable_collisions link1="${prefix}rg2_l_finger_link" link2="${prefix}rg2_l_truss_arm_link" reason="Adjacent" />
+      <disable_collisions link1="${prefix}rg2_r_moment_arm_link" link2="${prefix}rg2_r_finger_link" reason="Adjacent" />
+      <disable_collisions link1="${prefix}rg2_r_finger_link" link2="${prefix}rg2_r_truss_arm_link" reason="Adjacent" />
+      <disable_collisions link1="${prefix}rg2_l_finger_link" link2="${prefix}rg2_r_finger_link" reason="Never" />
+      <disable_collisions link1="${prefix}rg2_l_finger_link" link2="${prefix}rg2_r_moment_arm_link" reason="Never" />
+      <disable_collisions link1="${prefix}rg2_l_finger_link" link2="${prefix}rg2_r_truss_arm_link" reason="Never" />
+      <disable_collisions link1="${prefix}rg2_r_finger_link" link2="${prefix}rg2_l_moment_arm_link" reason="Never" />
+      <disable_collisions link1="${prefix}rg2_r_finger_link" link2="${prefix}rg2_l_truss_arm_link" reason="Never" />
+      <disable_collisions link1="${prefix}rg2_l_moment_arm_link" link2="${prefix}rg2_r_moment_arm_link" reason="Never" />
+      <disable_collisions link1="${prefix}rg2_l_moment_arm_link" link2="${prefix}rg2_r_truss_arm_link" reason="Never" />
+      <disable_collisions link1="${prefix}rg2_r_moment_arm_link" link2="${prefix}rg2_l_truss_arm_link" reason="Never" />
+      <disable_collisions link1="${prefix}rg2_l_truss_arm_link" link2="${prefix}rg2_r_truss_arm_link" reason="Never" />
+      <disable_collisions link1="${prefix}rg2_l_moment_arm_link" link2="${prefix}rg2_l_truss_arm_link" reason="Never" />
+      <disable_collisions link1="${prefix}rg2_r_moment_arm_link" link2="${prefix}rg2_r_truss_arm_link" reason="Never" />
+    </xacro:if>
   </xacro:macro>
 </robot>
